File: power_reg.kicad_sch (KiCad schematic)
At the start: 7 parts, among them U2 TPS561201DDCR

Commit message: feat: populate all jlcpcb part#
Parts:
- C10: Part C388001 -> C14663
- C7, C8: Part (none) -> C13585
- R1: value R -> 33.2K; Part (none) -> C4216
- R2: value R -> 10K; Part (none) -> C25804
Changed lines of the file:
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@@
+			)
+		)
+		(property "Part" "C13585"
+			(at 153.67 142.24 0)
+			(effects
+				(font
+					(size 1.27 1.27)
+				)
+				(hide yes)
 			)
 		)
@@
 			)
 		)
-		(property "Part" "C388001"
+		(property "Part" "C14663"
 			(at 166.37 86.36 90)
 			(effects
@@
 			)
 		)
-		(property "Value" "R"
+		(property "Value" "33.2K"
 			(at 187.96 93.9799 0)
 			(effects
@@
 			)
 		)
+		(property "Part" "C4216"
+			(at 185.42 92.71 0)
+			(effects
+				(font
+					(size 1.27 1.27)
+				)
+				(hide yes)
+			)
+		)
 		(pin "1"
 		)
@@
 			)
 		)
+		(property "Part" "C13585"
+			(at 140.97 142.24 0)
+			(effects
+				(font
+					(size 1.27 1.27)
+				)
+				(hide yes)
+			)
+		)
 		(pin "2"
 		)
@@
 			)
 		)
-		(property "Value" "R"
+		(property "Value" "10K"
 			(at 187.96 104.1399 0)
 			(effects
@@
 			(at 185.42 102.87 0)
 			(effects
+				(font
+					(size 1.27 1.27)
+				)
+				(hide yes)
+			)
+		)
+		(property "Part" "C25804"
+			(at 185.42 102.87 0)
+			(effects
